Commit message: renaming

File: hts_description/urdf/panda.urdf (robot description, URDF)
Before this commit: robot panda, 12 links, 11 joints
Links:
- removed link panda_link0
- removed link panda_link1
- removed link panda_link2
- removed link panda_link3
- removed link panda_link4
- removed link panda_link5
- removed link panda_link6
- removed link panda_link7
- removed link panda_link8
- added link fr3_link0; collision mesh filename=package://hts_description/meshes/collision/link0.stl; visual mesh filename=package://hts_description/meshes/visual/link0.dae
- added link fr3_link1; collision mesh filename=package://hts_description/meshes/collision/link1.stl; visual mesh filename=package://hts_description/meshes/visual/link1.dae
- added link fr3_link2; collision mesh filename=package://hts_description/meshes/collision/link2.stl; visual mesh filename=package://hts_description/meshes/visual/link2.dae
- added link fr3_link3; collision mesh filename=package://hts_description/meshes/collision/link3.stl; visual mesh filename=package://hts_description/meshes/visual/link3.dae
- added link fr3_link4; collision mesh filename=package://hts_description/meshes/collision/link4.stl; visual mesh filename=package://hts_description/meshes/visual/link4.dae
- added link fr3_link5; collision mesh filename=package://hts_description/meshes/collision/link5.stl; visual mesh filename=package://hts_description/meshes/visual/link5.dae
- added link fr3_link6; collision mesh filename=package://hts_description/meshes/collision/link6.stl; visual mesh filename=package://hts_description/meshes/visual/link6.dae
- added link fr3_link7; collision mesh filename=package://hts_description/meshes/collision/link7.stl; visual mesh filename=package://hts_description/meshes/visual/link7.dae
- added link fr3_link8
- link panda_hand: geometry collision mesh filename=package://hts_description/meshes/collision/hand.stl; visual mesh filename=package://hts_description/meshes/visual/hand.dae
- link panda_leftfinger: geometry collision mesh filename=package://hts_description/meshes/collision/finger.stl; visual mesh filename=package://hts_description/meshes/visual/finger.dae
- link panda_rightfinger: geometry collision mesh filename=package://hts_description/meshes/collision/finger.stl; visual mesh filename=package://hts_description/meshes/visual/finger.dae
Joints:
- removed joint panda_joint1
- removed joint panda_joint2
- removed joint panda_joint3
- removed joint panda_joint4
- removed joint panda_joint5
- removed joint panda_joint6
- removed joint panda_joint7
- removed joint panda_joint8
- added joint fr3_joint1: type revolute, parent fr3_link0, child fr3_link1, origin xyz=0 0 0.333 rpy=0 0 0, axis 0 0 1, limit lower=-2.9671 upper=2.9671 effort=87 velocity=2.3925
- added joint fr3_joint2: type revolute, parent fr3_link1, child fr3_link2, origin xyz=0 0 0 rpy=-1.57079632679 0 0, axis 0 0 1, limit lower=-1.8326 upper=1.8326 effort=87 velocity=2.3925
- added joint fr3_joint3: type revolute, parent fr3_link2, child fr3_link3, origin xyz=0 -0.316 0 rpy=1.57079632679 0 0, axis 0 0 1, limit lower=-2.9671 upper=2.9671 effort=87 velocity=2.3925
- added joint fr3_joint4: type revolute, parent fr3_link3, child fr3_link4, origin xyz=0.0825 0 0 rpy=1.57079632679 0 0, axis 0 0 1, limit lower=-3.1416 upper=0.0873 effort=87 velocity=2.3925
- added joint fr3_joint5: type revolute, parent fr3_link4, child fr3_link5, origin xyz=-0.0825 0.384 0 rpy=-1.57079632679 0 0, axis 0 0 1, limit lower=-2.9671 upper=2.9671 effort=12 velocity=2.8710
- added joint fr3_joint6: type revolute, parent fr3_link5, child fr3_link6, origin xyz=0 0 0 rpy=1.57079632679 0 0, axis 0 0 1, limit lower=-0.0873 upper=3.8223 effort=12 velocity=2.8710
- added joint fr3_joint7: type revolute, parent fr3_link6, child fr3_link7, origin xyz=0.088 0 0 rpy=1.57079632679 0 0, axis 0 0 1, limit lower=-2.9671 upper=2.9671 effort=12 velocity=2.8710
- added joint fr3_joint8: type fixed, parent fr3_link7, child fr3_link8, origin xyz=0 0 0.107 rpy=0 0 0, axis 0 0 0
- joint panda_hand_joint: parent panda_link8 -> fr3_link8

File: hts_description/urdf/panda.urdf.xacro (robot description, xacro)
@@ -5,13 +5,13 @@
 <!-- =================================================================================== -->
 <robot name="panda" xmlns:xacro="http://www.ros.org/wiki/xacro">
-    <link name="panda_link0">
-        <visual>
-            <geometry>
-                <mesh filename="file://$(find moveit_resources_panda_description)/meshes/visual/link0.dae" />
-            </geometry>
-        </visual>
-        <collision>
-            <geometry>
-                <mesh filename="file://$(find moveit_resources_panda_description)/meshes/collision/link0.stl" />
+    <link name="fr3_link0">
+        <visual>
+            <geometry>
+                <mesh filename="file://$(find hts_description)/meshes/visual/link0.dae" />
+            </geometry>
+        </visual>
+        <collision>
+            <geometry>
+                <mesh filename="file://$(find hts_description)/meshes/collision/link0.stl" />
             </geometry>
         </collision>
@@ -22,13 +22,13 @@
         </inertial>
     </link>
-    <link name="panda_link1">
-        <visual>
-            <geometry>
-                <mesh filename="file://$(find moveit_resources_panda_description)/meshes/visual/link1.dae" />
-            </geometry>
-        </visual>
-        <collision>
-            <geometry>
-                <mesh filename="file://$(find moveit_resources_panda_description)/meshes/collision/link1.stl" />
+    <link name="fr3_link1">
+        <visual>
+            <geometry>
+                <mesh filename="file://$(find hts_description)/meshes/visual/link1.dae" />
+            </geometry>
+        </visual>
+        <collision>
+            <geometry>
+                <mesh filename="file://$(find hts_description)/meshes/collision/link1.stl" />
             </geometry>
         </collision>
@@ -39,22 +39,22 @@
         </inertial>
     </link>
-    <joint name="panda_joint1" type="revolute">
+    <joint name="fr3_joint1" type="revolute">
         <safety_controller k_position="100.0" k_velocity="40.0" soft_lower_limit="-2.8973" soft_upper_limit="2.8973" />
         <origin rpy="0 0 0" xyz="0 0 0.333" />
-        <parent link="panda_link0" />
-        <child link="panda_link1" />
+        <parent link="fr3_link0" />
+        <child link="fr3_link1" />
         <axis xyz="0 0 1" />
         <limit effort="87" lower="-2.9671" upper="2.9671" velocity="2.3925" />
         <dynamics D="1" K="7000" damping="0.003" friction="0.0" mu_coulomb="0" mu_viscous="16" />
     </joint>
-    <link name="panda_link2">
-        <visual>
-            <geometry>
-                <mesh filename="file://$(find moveit_resources_panda_description)/meshes/visual/link2.dae" />
-            </geometry>
-        </visual>
-        <collision>
-            <geometry>
-                <mesh filename="file://$(find moveit_resources_panda_description)/meshes/collision/link2.stl" />
+    <link name="fr3_link2">
+        <visual>
+            <geometry>
+                <mesh filename="file://$(find hts_description)/meshes/visual/link2.dae" />
+            </geometry>
+        </visual>
+        <collision>
+            <geometry>
+                <mesh filename="file://$(find hts_description)/meshes/collision/link2.stl" />
             </geometry>
         </collision>
@@ -65,22 +65,22 @@
         </inertial>
     </link>
-    <joint name="panda_joint2" type="revolute">
+    <joint name="fr3_joint2" type="revolute">
         <safety_controller k_position="100.0" k_velocity="40.0" soft_lower_limit="-1.7628" soft_upper_limit="1.7628" />
         <origin rpy="-1.57079632679 0 0" xyz="0 0 0" />
-        <parent link="panda_link1" />
-        <child link="panda_link2" />
+        <parent link="fr3_link1" />
+        <child link="fr3_link2" />
         <axis xyz="0 0 1" />
         <limit effort="87" lower="-1.8326" upper="1.8326" velocity="2.3925" />
         <dynamics D="1" K="7000" damping="0.003" friction="0.0" mu_coulomb="0" mu_viscous="16" />
     </joint>
-    <link name="panda_link3">
-        <visual>
-            <geometry>
-                <mesh filename="file://$(find moveit_resources_panda_description)/meshes/visual/link3.dae" />
-            </geometry>
-        </visual>
-        <collision>
-            <geometry>
-                <mesh filename="file://$(find moveit_resources_panda_description)/meshes/collision/link3.stl" />
+    <link name="fr3_link3">
+        <visual>
+            <geometry>
+                <mesh filename="file://$(find hts_description)/meshes/visual/link3.dae" />
+            </geometry>
+        </visual>
+        <collision>
+            <geometry>
+                <mesh filename="file://$(find hts_description)/meshes/collision/link3.stl" />
             </geometry>
         </collision>
@@ -91,22 +91,22 @@
         </inertial>
     </link>
-    <joint name="panda_joint3" type="revolute">
+    <joint name="fr3_joint3" type="revolute">
         <safety_controller k_position="100.0" k_velocity="40.0" soft_lower_limit="-2.8973" soft_upper_limit="2.8973" />
         <origin rpy="1.57079632679 0 0" xyz="0 -0.316 0" />
-        <parent link="panda_link2" />
-        <child link="panda_link3" />
+        <parent link="fr3_link2" />
+        <child link="fr3_link3" />
         <axis xyz="0 0 1" />
         <limit effort="87" lower="-2.9671" upper="2.9671" velocity="2.3925" />
         <dynamics D="1" K="7000" damping="0.003" friction="0.0" mu_coulomb="0" mu_viscous="16" />
     </joint>
-    <link name="panda_link4">
-        <visual>
-            <geometry>
-                <mesh filename="file://$(find moveit_resources_panda_description)/meshes/visual/link4.dae" />
-            </geometry>
-        </visual>
-        <collision>
-            <geometry>
-                <mesh filename="file://$(find moveit_resources_panda_description)/meshes/collision/link4.stl" />
+    <link name="fr3_link4">
+        <visual>
+            <geometry>
+                <mesh filename="file://$(find hts_description)/meshes/visual/link4.dae" />
+            </geometry>
+        </visual>
+        <collision>
+            <geometry>
+                <mesh filename="file://$(find hts_description)/meshes/collision/link4.stl" />
             </geometry>
         </collision>
@@ -117,22 +117,22 @@
         </inertial>
     </link>
-    <joint name="panda_joint4" type="revolute">
+    <joint name="fr3_joint4" type="revolute">
         <safety_controller k_position="100.0" k_velocity="40.0" soft_lower_limit="-3.0718" soft_upper_limit="0.0175" />
         <origin rpy="1.57079632679 0 0" xyz="0.0825 0 0" />
-        <parent link="panda_link3" />
-        <child link="panda_link4" />
+        <parent link="fr3_link3" />
+        <child link="fr3_link4" />
         <axis xyz="0 0 1" />
         <limit effort="87" lower="-3.1416" upper="0.0873" velocity="2.3925" />
         <dynamics D="1" K="7000" damping="0.003" friction="0.0" mu_coulomb="0" mu_viscous="16" />
     </joint>
-    <link name="panda_link5">
-        <visual>
-            <geometry>
-                <mesh filename="file://$(find moveit_resources_panda_description)/meshes/visual/link5.dae" />
-            </geometry>
-        </visual>
-        <collision>
-            <geometry>
-                <mesh filename="file://$(find moveit_resources_panda_description)/meshes/collision/link5.stl" />
+    <link name="fr3_link5">
+        <visual>
+            <geometry>
+                <mesh filename="file://$(find hts_description)/meshes/visual/link5.dae" />
+            </geometry>
+        </visual>
+        <collision>
+            <geometry>
+                <mesh filename="file://$(find hts_description)/meshes/collision/link5.stl" />
             </geometry>
         </collision>
@@ -143,22 +143,22 @@
         </inertial>
     </link>
-    <joint name="panda_joint5" type="revolute">
+    <joint name="fr3_joint5" type="revolute">
         <safety_controller k_position="100.0" k_velocity="40.0" soft_lower_limit="-2.8973" soft_upper_limit="2.8973" />
         <origin rpy="-1.57079632679 0 0" xyz="-0.0825 0.384 0" />
-        <parent link="panda_link4" />
-        <child link="panda_link5" />
+        <parent link="fr3_link4" />
+        <child link="fr3_link5" />
         <axis xyz="0 0 1" />
         <limit effort="12" lower="-2.9671" upper="2.9671" velocity="2.8710" />
         <dynamics D="1" K="7000" damping="0.003" friction="0.0" mu_coulomb="0" mu_viscous="16" />
     </joint>
-    <link name="panda_link6">
-        <visual>
-            <geometry>
-                <mesh filename="file://$(find moveit_resources_panda_description)/meshes/visual/link6.dae" />
-            </geometry>
-        </visual>
-        <collision>
-            <geometry>
-                <mesh filename="file://$(find moveit_resources_panda_description)/meshes/collision/link6.stl" />
+    <link name="fr3_link6">
+        <visual>
+            <geometry>
+                <mesh filename="file://$(find hts_description)/meshes/visual/link6.dae" />
+            </geometry>
+        </visual>
+        <collision>
+            <geometry>
+                <mesh filename="file://$(find hts_description)/meshes/collision/link6.stl" />
             </geometry>
         </collision>
@@ -169,22 +169,22 @@
         </inertial>
     </link>
-    <joint name="panda_joint6" type="revolute">
+    <joint name="fr3_joint6" type="revolute">
         <safety_controller k_position="100.0" k_velocity="40.0" soft_lower_limit="-0.0175" soft_upper_limit="3.7525" />
         <origin rpy="1.57079632679 0 0" xyz="0 0 0" />
-        <parent link="panda_link5" />
-        <child link="panda_link6" />
+        <parent link="fr3_link5" />
+        <child link="fr3_link6" />
         <axis xyz="0 0 1" />
         <limit effort="12" lower="-0.0873" upper="3.8223" velocity="2.8710" />
         <dynamics D="1" K="7000" damping="0.003" friction="0.0" mu_coulomb="0" mu_viscous="16" />
     </joint>
-    <link name="panda_link7">
-        <visual>
-            <geometry>
-                <mesh filename="file://$(find moveit_resources_panda_description)/meshes/visual/link7.dae" />
-            </geometry>
-        </visual>
-        <collision>
-            <geometry>
-                <mesh filename="file://$(find moveit_resources_panda_description)/meshes/collision/link7.stl" />
+    <link name="fr3_link7">
+        <visual>
+            <geometry>
+                <mesh filename="file://$(find hts_description)/meshes/visual/link7.dae" />
+            </geometry>
+        </visual>
+        <collision>
+            <geometry>
+                <mesh filename="file://$(find hts_description)/meshes/collision/link7.stl" />
             </geometry>
         </collision>
@@ -195,22 +195,22 @@
         </inertial>
     </link>
-    <joint name="panda_joint7" type="revolute">
+    <joint name="fr3_joint7" type="revolute">
         <safety_controller k_position="100.0" k_velocity="40.0" soft_lower_limit="-2.8973" soft_upper_limit="2.8973" />
         <origin rpy="1.57079632679 0 0" xyz="0.088 0 0" />
-        <parent link="panda_link6" />
-        <child link="panda_link7" />
+        <parent link="fr3_link6" />
+        <child link="fr3_link7" />
         <axis xyz="0 0 1" />
         <limit effort="12" lower="-2.9671" upper="2.9671" velocity="2.8710" />
         <dynamics D="1" K="7000" damping="0.003" friction="0.0" mu_coulomb="0" mu_viscous="16" />
     </joint>
-    <link name="panda_link8" />
-    <joint name="panda_joint8" type="fixed">
+    <link name="fr3_link8" />
+    <joint name="fr3_joint8" type="fixed">
         <origin rpy="0 0 0" xyz="0 0 0.107" />
-        <parent link="panda_link7" />
-        <child link="panda_link8" />
+        <parent link="fr3_link7" />
+        <child link="fr3_link8" />
         <axis xyz="0 0 0" />
     </joint>
     <joint name="panda_hand_joint" type="fixed">
-        <parent link="panda_link8" />
+        <parent link="fr3_link8" />
         <child link="panda_hand" />
         <origin rpy="0 0 -0.785398163397" xyz="0 0 0" />
@@ -219,10 +219,10 @@
         <visual>
             <geometry>
-                <mesh filename="file://$(find moveit_resources_panda_description)/meshes/visual/hand.dae" />
-            </geometry>
-        </visual>
-        <collision>
-            <geometry>
-                <mesh filename="file://$(find moveit_resources_panda_description)/meshes/collision/hand.stl" />
+                <mesh filename="file://$(find hts_description)/meshes/visual/hand.dae" />
+            </geometry>
+        </visual>
+        <collision>
+            <geometry>
+                <mesh filename="file://$(find hts_description)/meshes/collision/hand.stl" />
             </geometry>
         </collision>
@@ -236,10 +236,10 @@
         <visual>
             <geometry>
-                <mesh filename="file://$(find moveit_resources_panda_description)/meshes/visual/finger.dae" />
-            </geometry>
-        </visual>
-        <collision>
-            <geometry>
-                <mesh filename="file://$(find moveit_resources_panda_description)/meshes/collision/finger.stl" />
+                <mesh filename="file://$(find hts_description)/meshes/visual/finger.dae" />
+            </geometry>
+        </visual>
+        <collision>
+            <geometry>
+                <mesh filename="file://$(find hts_description)/meshes/collision/finger.stl" />
             </geometry>
         </collision>
@@ -254,5 +254,5 @@
             <origin rpy="0 0 3.14159265359" xyz="0 0 0" />
             <geometry>
-                <mesh filename="file://$(find moveit_resources_panda_description)/meshes/visual/finger.dae" />
+                <mesh filename="file://$(find hts_description)/meshes/visual/finger.dae" />
             </geometry>
         </visual>
@@ -260,5 +260,5 @@
             <origin rpy="0 0 3.14159265359" xyz="0 0 0" />
             <geometry>
-                <mesh filename="file://$(find moveit_resources_panda_description)/meshes/collision/finger.stl" />
+                <mesh filename="file://$(find hts_description)/meshes/collision/finger.stl" />
             </geometry>
         </collision>

File: hts_moveit_config/config/panda.ros2_control.xacro (robot description, xacro)
@@ -14,8 +14,8 @@
                 </xacro:if>
             </hardware>
-            <joint name="panda_joint1">
+            <joint name="fr3_joint1">
                 <command_interface name="position"/>
                 <state_interface name="position">
-                  <param name="initial_value">${initial_positions['panda_joint1']}</param>
+                  <param name="initial_value">${initial_positions['fr3_joint1']}</param>
                 </state_interface>
                 <state_interface name="velocity">
@@ -23,8 +23,8 @@
                 </state_interface>
             </joint>
-            <joint name="panda_joint2">
+            <joint name="fr3_joint2">
                 <command_interface name="position"/>
                 <state_interface name="position">
-                  <param name="initial_value">${initial_positions['panda_joint2']}</param>
+                  <param name="initial_value">${initial_positions['fr3_joint2']}</param>
                 </state_interface>
                 <state_interface name="velocity">
@@ -32,8 +32,8 @@
                 </state_interface>
             </joint>
-            <joint name="panda_joint3">
+            <joint name="fr3_joint3">
                 <command_interface name="position"/>
                 <state_interface name="position">
-                  <param name="initial_value">${initial_positions['panda_joint3']}</param>
+                  <param name="initial_value">${initial_positions['fr3_joint3']}</param>
                 </state_interface>
                 <state_interface name="velocity">
@@ -41,8 +41,8 @@
                 </state_interface>
             </joint>
-            <joint name="panda_joint4">
+            <joint name="fr3_joint4">
                 <command_interface name="position"/>
                 <state_interface name="position">
-                  <param name="initial_value">${initial_positions['panda_joint4']}</param>
+                  <param name="initial_value">${initial_positions['fr3_joint4']}</param>
                 </state_interface>
                 <state_interface name="velocity">
@@ -50,8 +50,8 @@
                 </state_interface>
             </joint>
-            <joint name="panda_joint5">
+            <joint name="fr3_joint5">
                 <command_interface name="position"/>
                 <state_interface name="position">
-                  <param name="initial_value">${initial_positions['panda_joint5']}</param>
+                  <param name="initial_value">${initial_positions['fr3_joint5']}</param>
                 </state_interface>
                 <state_interface name="velocity">
@@ -59,8 +59,8 @@
                 </state_interface>
             </joint>
-            <joint name="panda_joint6">
+            <joint name="fr3_joint6">
                 <command_interface name="position"/>
                 <state_interface name="position">
-                  <param name="initial_value">${initial_positions['panda_joint6']}</param>
+                  <param name="initial_value">${initial_positions['fr3_joint6']}</param>
                 </state_interface>
                 <state_interface name="velocity">
@@ -68,8 +68,8 @@
                 </state_interface>
             </joint>
-            <joint name="panda_joint7">
+            <joint name="fr3_joint7">
                 <command_interface name="position"/>
                 <state_interface name="position">
-                  <param name="initial_value">${initial_positions['panda_joint7']}</param>
+                  <param name="initial_value">${initial_positions['fr3_joint7']}</param>
                 </state_interface>
                 <state_interface name="velocity">

File: hts_moveit_config/config/panda.urdf.xacro (robot description, xacro)
@@ -4,5 +4,5 @@
     <xacro:arg name="ros2_control_hardware_type" default="mock_components" />
     <!-- Import panda urdf file -->
-    <xacro:include filename="$(find moveit_resources_panda_description)/urdf/panda.urdf.xacro" />
+    <xacro:include filename="$(find hts_description)/urdf/panda.urdf.xacro" />
     <!-- Import panda ros2_control description -->
     <xacro:include filename="panda.ros2_control.xacro" />
