Commit message: renaming

File: hts_moveit_config/config/panda_arm.xacro (robot description, xacro)
@@ -8,57 +8,57 @@
     <!--SUBGROUPS: Groups can also be formed by referencing to already defined group names-->
     <group name="panda_arm">
-      <chain base_link="panda_link0" tip_link="panda_link8" />
+      <chain base_link="fr3_link0" tip_link="fr3_link8" />
     </group>
     <!--GROUP STATES: Purpose: Define a named state for a particular group, in terms of joint values. This is useful to define states like 'folded arms'-->
     <group_state name="ready" group="panda_arm">
-      <joint name="panda_joint1" value="0" />
-      <joint name="panda_joint2" value="-0.785" />
-      <joint name="panda_joint3" value="0" />
-      <joint name="panda_joint4" value="-2.356" />
-      <joint name="panda_joint5" value="0" />
-      <joint name="panda_joint6" value="1.571" />
-      <joint name="panda_joint7" value="0.785" />
+      <joint name="fr3_joint1" value="0" />
+      <joint name="fr3_joint2" value="-0.785" />
+      <joint name="fr3_joint3" value="0" />
+      <joint name="fr3_joint4" value="-2.356" />
+      <joint name="fr3_joint5" value="0" />
+      <joint name="fr3_joint6" value="1.571" />
+      <joint name="fr3_joint7" value="0.785" />
     </group_state>
     <group_state name="extended" group="panda_arm">
-      <joint name="panda_joint1" value="0" />
-      <joint name="panda_joint2" value="0" />
-      <joint name="panda_joint3" value="0" />
-      <joint name="panda_joint4" value="0" />
-      <joint name="panda_joint5" value="0" />
-      <joint name="panda_joint6" value="1.571" />
-      <joint name="panda_joint7" value="0.785" />
+      <joint name="fr3_joint1" value="0" />
+      <joint name="fr3_joint2" value="0" />
+      <joint name="fr3_joint3" value="0" />
+      <joint name="fr3_joint4" value="0" />
+      <joint name="fr3_joint5" value="0" />
+      <joint name="fr3_joint6" value="1.571" />
+      <joint name="fr3_joint7" value="0.785" />
     </group_state>
     <group_state name="transport" group="panda_arm">
-      <joint name="panda_joint1" value="0" />
-      <joint name="panda_joint2" value="-0.5599" />
-      <joint name="panda_joint3" value="0" />
-      <joint name="panda_joint4" value="-2.97" />
-      <joint name="panda_joint5" value="0" />
-      <joint name="panda_joint6" value="0" />
-      <joint name="panda_joint7" value="0.785" />
+      <joint name="fr3_joint1" value="0" />
+      <joint name="fr3_joint2" value="-0.5599" />
+      <joint name="fr3_joint3" value="0" />
+      <joint name="fr3_joint4" value="-2.97" />
+      <joint name="fr3_joint5" value="0" />
+      <joint name="fr3_joint6" value="0" />
+      <joint name="fr3_joint7" value="0.785" />
     </group_state>
     <!--END EFFECTOR: Purpose: Represent information about an end effector.-->
     <!--VIRTUAL JOINT: Purpose: this element defines a virtual joint between a robot link and an external frame of reference (considered fixed with respect to the robot)-->
-    <virtual_joint name="virtual_joint" type="floating" parent_frame="world" child_link="panda_link0" />
+    <virtual_joint name="virtual_joint" type="floating" parent_frame="world" child_link="fr3_link0" />
     <!--DISABLE COLLISIONS: By default it is assumed that any link of the robot could potentially come into collision with any other link in the robot. This tag disables collision checking between a specified pair of links. -->
-    <disable_collisions link1="panda_link0" link2="panda_link1" reason="Adjacent" />
-    <disable_collisions link1="panda_link0" link2="panda_link2" reason="Never" />
-    <disable_collisions link1="panda_link0" link2="panda_link3" reason="Never" />
-    <disable_collisions link1="panda_link0" link2="panda_link4" reason="Never" />
-    <disable_collisions link1="panda_link1" link2="panda_link2" reason="Adjacent" />
-    <disable_collisions link1="panda_link1" link2="panda_link3" reason="Never" />
-    <disable_collisions link1="panda_link1" link2="panda_link4" reason="Never" />
-    <disable_collisions link1="panda_link2" link2="panda_link3" reason="Adjacent" />
-    <disable_collisions link1="panda_link2" link2="panda_link4" reason="Never" />
-    <disable_collisions link1="panda_link2" link2="panda_link6" reason="Never" />
-    <disable_collisions link1="panda_link3" link2="panda_link4" reason="Adjacent" />
-    <disable_collisions link1="panda_link3" link2="panda_link5" reason="Never" />
-    <disable_collisions link1="panda_link3" link2="panda_link6" reason="Never" />
-    <disable_collisions link1="panda_link3" link2="panda_link7" reason="Never" />
-    <disable_collisions link1="panda_link4" link2="panda_link5" reason="Adjacent" />
-    <disable_collisions link1="panda_link4" link2="panda_link6" reason="Never" />
-    <disable_collisions link1="panda_link4" link2="panda_link7" reason="Never" />
-    <disable_collisions link1="panda_link5" link2="panda_link6" reason="Adjacent" />
-    <disable_collisions link1="panda_link6" link2="panda_link7" reason="Adjacent" />
+    <disable_collisions link1="fr3_link0" link2="fr3_link1" reason="Adjacent" />
+    <disable_collisions link1="fr3_link0" link2="fr3_link2" reason="Never" />
+    <disable_collisions link1="fr3_link0" link2="fr3_link3" reason="Never" />
+    <disable_collisions link1="fr3_link0" link2="fr3_link4" reason="Never" />
+    <disable_collisions link1="fr3_link1" link2="fr3_link2" reason="Adjacent" />
+    <disable_collisions link1="fr3_link1" link2="fr3_link3" reason="Never" />
+    <disable_collisions link1="fr3_link1" link2="fr3_link4" reason="Never" />
+    <disable_collisions link1="fr3_link2" link2="fr3_link3" reason="Adjacent" />
+    <disable_collisions link1="fr3_link2" link2="fr3_link4" reason="Never" />
+    <disable_collisions link1="fr3_link2" link2="fr3_link6" reason="Never" />
+    <disable_collisions link1="fr3_link3" link2="fr3_link4" reason="Adjacent" />
+    <disable_collisions link1="fr3_link3" link2="fr3_link5" reason="Never" />
+    <disable_collisions link1="fr3_link3" link2="fr3_link6" reason="Never" />
+    <disable_collisions link1="fr3_link3" link2="fr3_link7" reason="Never" />
+    <disable_collisions link1="fr3_link4" link2="fr3_link5" reason="Adjacent" />
+    <disable_collisions link1="fr3_link4" link2="fr3_link6" reason="Never" />
+    <disable_collisions link1="fr3_link4" link2="fr3_link7" reason="Never" />
+    <disable_collisions link1="fr3_link5" link2="fr3_link6" reason="Adjacent" />
+    <disable_collisions link1="fr3_link6" link2="fr3_link7" reason="Adjacent" />
   </xacro:macro>
 </robot>

File: hts_moveit_config/config/panda_arm_hand.srdf.xacro (robot description, xacro)
@@ -27,17 +27,17 @@
   </group_state>
   <!--END EFFECTOR: Purpose: Represent information about an end effector.-->
-  <end_effector name="hand" parent_link="panda_link8" group="hand" parent_group="panda_arm" />
+  <end_effector name="hand" parent_link="fr3_link8" group="hand" parent_group="panda_arm" />
   <!--DISABLE COLLISIONS: By default it is assumed that any link of the robot could potentially come into collision with any other link in the robot. This tag disables collision checking between a specified pair of links. -->
-  <disable_collisions link1="panda_hand" link2="panda_link3" reason="Never" />
-  <disable_collisions link1="panda_hand" link2="panda_link4" reason="Never" />
-  <disable_collisions link1="panda_hand" link2="panda_link6" reason="Never" />
-  <disable_collisions link1="panda_hand" link2="panda_link7" reason="Adjacent" />
-  <disable_collisions link1="panda_leftfinger" link2="panda_link3" reason="Never" />
-  <disable_collisions link1="panda_leftfinger" link2="panda_link4" reason="Never" />
-  <disable_collisions link1="panda_leftfinger" link2="panda_link6" reason="Never" />
-  <disable_collisions link1="panda_leftfinger" link2="panda_link7" reason="Never" />
-  <disable_collisions link1="panda_link3" link2="panda_rightfinger" reason="Never" />
-  <disable_collisions link1="panda_link4" link2="panda_rightfinger" reason="Never" />
-  <disable_collisions link1="panda_link6" link2="panda_rightfinger" reason="Never" />
-  <disable_collisions link1="panda_link7" link2="panda_rightfinger" reason="Never" />
+  <disable_collisions link1="panda_hand" link2="fr3_link3" reason="Never" />
+  <disable_collisions link1="panda_hand" link2="fr3_link4" reason="Never" />
+  <disable_collisions link1="panda_hand" link2="fr3_link6" reason="Never" />
+  <disable_collisions link1="panda_hand" link2="fr3_link7" reason="Adjacent" />
+  <disable_collisions link1="panda_leftfinger" link2="fr3_link3" reason="Never" />
+  <disable_collisions link1="panda_leftfinger" link2="fr3_link4" reason="Never" />
+  <disable_collisions link1="panda_leftfinger" link2="fr3_link6" reason="Never" />
+  <disable_collisions link1="panda_leftfinger" link2="fr3_link7" reason="Never" />
+  <disable_collisions link1="fr3_link3" link2="panda_rightfinger" reason="Never" />
+  <disable_collisions link1="fr3_link4" link2="panda_rightfinger" reason="Never" />
+  <disable_collisions link1="fr3_link6" link2="panda_rightfinger" reason="Never" />
+  <disable_collisions link1="fr3_link7" link2="panda_rightfinger" reason="Never" />
 </robot>

Commit message: more renaming

File: hts_description/urdf/panda.urdf (robot description, URDF)
Before this commit: robot panda, 12 links, 11 joints
Links:
- removed link panda_hand
- added link fr3_hand; collision mesh filename=package://hts_description/meshes/collision/hand.stl; visual mesh filename=package://hts_description/meshes/visual/hand.dae
Joints:
- removed joint panda_finger_joint1
- removed joint panda_finger_joint2
- removed joint panda_hand_joint
- added joint fr3_finger_joint1: type prismatic, parent fr3_hand, child panda_leftfinger, origin xyz=0 0 0.0584 rpy=0 0 0, axis 0 1 0, limit lower=0.0 upper=0.04 effort=20 velocity=0.2
- added joint fr3_finger_joint2: type prismatic, parent fr3_hand, child panda_rightfinger, origin xyz=0 0 0.0584 rpy=0 0 0, axis 0 -1 0, limit lower=0.0 upper=0.04 effort=20 velocity=0.2, mimic joint=fr3_finger_joint1
- added joint fr3_hand_joint: type fixed, parent fr3_link8, child fr3_hand, origin xyz=0 0 0 rpy=0 0 -0.785398163397

File: hts_description/urdf/panda.urdf.xacro (robot description, xacro)
@@ -211,10 +211,10 @@
         <axis xyz="0 0 0" />
     </joint>
-    <joint name="panda_hand_joint" type="fixed">
+    <joint name="fr3_hand_joint" type="fixed">
         <parent link="fr3_link8" />
-        <child link="panda_hand" />
+        <child link="fr3_hand" />
         <origin rpy="0 0 -0.785398163397" xyz="0 0 0" />
     </joint>
-    <link name="panda_hand">
+    <link name="fr3_hand">
         <visual>
             <geometry>
@@ -269,6 +269,6 @@
         </inertial>
     </link>
-    <joint name="panda_finger_joint1" type="prismatic">
-        <parent link="panda_hand" />
+    <joint name="fr3_finger_joint1" type="prismatic">
+        <parent link="fr3_hand" />
         <child link="panda_leftfinger" />
         <origin rpy="0 0 0" xyz="0 0 0.0584" />
@@ -277,11 +277,11 @@
         <dynamics damping="0.3" />
     </joint>
-    <joint name="panda_finger_joint2" type="prismatic">
-        <parent link="panda_hand" />
+    <joint name="fr3_finger_joint2" type="prismatic">
+        <parent link="fr3_hand" />
         <child link="panda_rightfinger" />
         <origin rpy="0 0 0" xyz="0 0 0.0584" />
         <axis xyz="0 -1 0" />
         <limit effort="20" lower="0.0" upper="0.04" velocity="0.2" />
-        <mimic joint="panda_finger_joint1" />
+        <mimic joint="fr3_finger_joint1" />
         <dynamics damping="0.3" />
     </joint>

File: hts_moveit_config/config/fr3_arm.srdf.xacro (robot description, xacro)
@@ -5,5 +5,5 @@
 -->
 <robot xmlns:xacro="http://www.ros.org/wiki/xacro" name="panda">
-  <xacro:include filename="$(find moveit_resources_panda_moveit_config)/config/panda_arm.xacro" />
-  <xacro:panda_arm />
+  <xacro:include filename="$(find moveit_resources_panda_moveit_config)/config/fr3_arm.xacro" />
+  <xacro:fr3_arm />
 </robot>

File: hts_moveit_config/config/fr3_arm.xacro (robot description, xacro)
@@ -1,5 +1,5 @@
 <?xml version="1.0" ?>
 <robot xmlns:xacro="http://www.ros.org/wiki/xacro" name="panda">
-  <xacro:macro name="panda_arm">
+  <xacro:macro name="fr3_arm">
     <!--GROUPS: Representation of a set of joints and links. This can be useful for specifying DOF to plan for, defining arms, end effectors, etc-->
     <!--LINKS: When a link is specified, the parent joint of that link (if it exists) is automatically included-->
@@ -7,9 +7,9 @@
     <!--CHAINS: When a chain is specified, all the links along the chain (including endpoints) are included in the group. Additionally, all the joints that are parents to included links are also included. This means that joints along the chain and the parent joint of the base link are included in the group-->
     <!--SUBGROUPS: Groups can also be formed by referencing to already defined group names-->
-    <group name="panda_arm">
+    <group name="fr3_arm">
       <chain base_link="fr3_link0" tip_link="fr3_link8" />
     </group>
     <!--GROUP STATES: Purpose: Define a named state for a particular group, in terms of joint values. This is useful to define states like 'folded arms'-->
-    <group_state name="ready" group="panda_arm">
+    <group_state name="ready" group="fr3_arm">
       <joint name="fr3_joint1" value="0" />
       <joint name="fr3_joint2" value="-0.785" />
@@ -20,5 +20,5 @@
       <joint name="fr3_joint7" value="0.785" />
     </group_state>
-    <group_state name="extended" group="panda_arm">
+    <group_state name="extended" group="fr3_arm">
       <joint name="fr3_joint1" value="0" />
       <joint name="fr3_joint2" value="0" />
@@ -29,5 +29,5 @@
       <joint name="fr3_joint7" value="0.785" />
     </group_state>
-    <group_state name="transport" group="panda_arm">
+    <group_state name="transport" group="fr3_arm">
       <joint name="fr3_joint1" value="0" />
       <joint name="fr3_joint2" value="-0.5599" />

File: hts_moveit_config/config/fr3_arm_hand.srdf.xacro (robot description, xacro)
@@ -5,7 +5,7 @@
 -->
 <robot xmlns:xacro="http://www.ros.org/wiki/xacro" name="panda">
-  <xacro:include filename="$(find moveit_resources_panda_moveit_config)/config/panda_arm.xacro" />
+  <xacro:include filename="$(find moveit_resources_panda_moveit_config)/config/fr3_arm.xacro" />
   <xacro:include filename="$(find moveit_resources_panda_moveit_config)/config/hand.xacro" />
-  <xacro:panda_arm />
+  <xacro:fr3_arm />
   <xacro:hand />
   <!--GROUPS: Representation of a set of joints and links. This can be useful for specifying DOF to plan for, defining arms, end effectors, etc-->
@@ -14,23 +14,23 @@
   <!--CHAINS: When a chain is specified, all the links along the chain (including endpoints) are included in the group. Additionally, all the joints that are parents to included links are also included. This means that joints along the chain and the parent joint of the base link are included in the group-->
   <!--SUBGROUPS: Groups can also be formed by referencing to already defined group names-->
-  <group name="panda_arm_hand">
-    <group name="panda_arm" />
+  <group name="fr3_arm_hand">
+    <group name="fr3_arm" />
     <group name="hand" />
   </group>
   <group_state name="open" group="hand">
-    <joint name="panda_finger_joint1" value="0.035" />
-    <joint name="panda_finger_joint2" value="0.035" />
+    <joint name="fr3_finger_joint1" value="0.035" />
+    <joint name="fr3_finger_joint2" value="0.035" />
   </group_state>
   <group_state name="close" group="hand">
-    <joint name="panda_finger_joint1" value="0" />
-    <joint name="panda_finger_joint2" value="0" />
+    <joint name="fr3_finger_joint1" value="0" />
+    <joint name="fr3_finger_joint2" value="0" />
   </group_state>
   <!--END EFFECTOR: Purpose: Represent information about an end effector.-->
-  <end_effector name="hand" parent_link="fr3_link8" group="hand" parent_group="panda_arm" />
+  <end_effector name="hand" parent_link="fr3_link8" group="hand" parent_group="fr3_arm" />
   <!--DISABLE COLLISIONS: By default it is assumed that any link of the robot could potentially come into collision with any other link in the robot. This tag disables collision checking between a specified pair of links. -->
-  <disable_collisions link1="panda_hand" link2="fr3_link3" reason="Never" />
-  <disable_collisions link1="panda_hand" link2="fr3_link4" reason="Never" />
-  <disable_collisions link1="panda_hand" link2="fr3_link6" reason="Never" />
-  <disable_collisions link1="panda_hand" link2="fr3_link7" reason="Adjacent" />
+  <disable_collisions link1="fr3_hand" link2="fr3_link3" reason="Never" />
+  <disable_collisions link1="fr3_hand" link2="fr3_link4" reason="Never" />
+  <disable_collisions link1="fr3_hand" link2="fr3_link6" reason="Never" />
+  <disable_collisions link1="fr3_hand" link2="fr3_link7" reason="Adjacent" />
   <disable_collisions link1="panda_leftfinger" link2="fr3_link3" reason="Never" />
   <disable_collisions link1="panda_leftfinger" link2="fr3_link4" reason="Never" />

File: hts_moveit_config/config/fr3_hand.ros2_control.xacro (robot description, xacro)
@@ -1,5 +1,5 @@
 <?xml version="1.0"?>
 <robot xmlns:xacro="http://www.ros.org/wiki/xacro">
-    <xacro:macro name="panda_hand_ros2_control" params="name ros2_control_hardware_type">
+    <xacro:macro name="fr3_hand_ros2_control" params="name ros2_control_hardware_type">
         <ros2_control name="${name}" type="system">
             <hardware>
@@ -13,5 +13,5 @@
                 </xacro:if>
             </hardware>
-            <joint name="panda_finger_joint1">
+            <joint name="fr3_finger_joint1">
                 <command_interface name="position" />
                 <state_interface name="position">
@@ -22,5 +22,5 @@
                 </state_interface>
             </joint>
-            <joint name="panda_finger_joint2">
+            <joint name="fr3_finger_joint2">
                 <state_interface name="position">
                   <param name="initial_value">0.0</param>

File: hts_moveit_config/config/hand.xacro (robot description, xacro)
@@ -8,15 +8,15 @@
     <!--SUBGROUPS: Groups can also be formed by referencing to already defined group names-->
     <group name="hand">
-      <link name="panda_hand" />
+      <link name="fr3_hand" />
       <link name="panda_leftfinger" />
       <link name="panda_rightfinger" />
-      <joint name="panda_finger_joint1" />
-      <passive_joint name="panda_finger_joint2" />
+      <joint name="fr3_finger_joint1" />
+      <passive_joint name="fr3_finger_joint2" />
     </group>
     <!--GROUP STATES: Purpose: Define a named state for a particular group, in terms of joint values. This is useful to define states like 'folded arms'-->
     <!--END EFFECTOR: Purpose: Represent information about an end effector.-->
     <!--DISABLE COLLISIONS: By default it is assumed that any link of the robot could potentially come into collision with any other link in the robot. This tag disables collision checking between a specified pair of links. -->
-    <disable_collisions link1="panda_hand" link2="panda_leftfinger" reason="Adjacent" />
-    <disable_collisions link1="panda_hand" link2="panda_rightfinger" reason="Adjacent" />
+    <disable_collisions link1="fr3_hand" link2="panda_leftfinger" reason="Adjacent" />
+    <disable_collisions link1="fr3_hand" link2="panda_rightfinger" reason="Adjacent" />
     <disable_collisions link1="panda_leftfinger" link2="panda_rightfinger" reason="Default" />
   </xacro:macro>

File: hts_moveit_config/config/panda.urdf.xacro (robot description, xacro)
@@ -7,6 +7,6 @@
     <!-- Import panda ros2_control description -->
     <xacro:include filename="panda.ros2_control.xacro" />
-    <xacro:include filename="panda_hand.ros2_control.xacro" />
+    <xacro:include filename="fr3_hand.ros2_control.xacro" />
     <xacro:panda_ros2_control name="PandaFakeSystem" initial_positions_file="$(arg initial_positions_file)" ros2_control_hardware_type="$(arg ros2_control_hardware_type)"/>
-    <xacro:panda_hand_ros2_control name="PandaHandFakeSystem" ros2_control_hardware_type="$(arg ros2_control_hardware_type)"/>
+    <xacro:fr3_hand_ros2_control name="PandaHandFakeSystem" ros2_control_hardware_type="$(arg ros2_control_hardware_type)"/>
 </robot>
