Commit message: more renaming

File: hts_description/urdf/fr3.urdf (robot description, URDF)
Before this commit: robot panda, 12 links, 11 joints
Links:
- removed link panda_leftfinger
- removed link panda_rightfinger
- added link fr3_leftfinger; collision mesh filename=package://hts_description/meshes/collision/finger.stl; visual mesh filename=package://hts_description/meshes/visual/finger.dae
- added link fr3_rightfinger; collision mesh filename=package://hts_description/meshes/collision/finger.stl; visual mesh filename=package://hts_description/meshes/visual/finger.dae
Joints:
- joint fr3_finger_joint1: child panda_leftfinger -> fr3_leftfinger
- joint fr3_finger_joint2: child panda_rightfinger -> fr3_rightfinger

File: hts_description/urdf/fr3.urdf.xacro (robot description, xacro)
@@ -1,5 +1,5 @@
 <?xml version="1.0" ?>
 <!-- =================================================================================== -->
-<!-- |    This document was autogenerated by xacro from /opt/ros/kinetic/share/moveit_resources/panda_description/urdf/panda.urdf | -->
+<!-- |    This document was autogenerated by xacro from /opt/ros/kinetic/share/moveit_resources/fr3_description/urdf/fr3.urdf | -->
 <!-- |    EDITING THIS FILE BY HAND IS NOT RECOMMENDED                                 | -->
 <!-- =================================================================================== -->
@@ -233,5 +233,5 @@
         </inertial>
     </link>
-    <link name="panda_leftfinger">
+    <link name="fr3_leftfinger">
         <visual>
             <geometry>
@@ -250,5 +250,5 @@
         </inertial>
     </link>
-    <link name="panda_rightfinger">
+    <link name="fr3_rightfinger">
         <visual>
             <origin rpy="0 0 3.14159265359" xyz="0 0 0" />
@@ -271,5 +271,5 @@
     <joint name="fr3_finger_joint1" type="prismatic">
         <parent link="fr3_hand" />
-        <child link="panda_leftfinger" />
+        <child link="fr3_leftfinger" />
         <origin rpy="0 0 0" xyz="0 0 0.0584" />
         <axis xyz="0 1 0" />
@@ -279,5 +279,5 @@
     <joint name="fr3_finger_joint2" type="prismatic">
         <parent link="fr3_hand" />
-        <child link="panda_rightfinger" />
+        <child link="fr3_rightfinger" />
         <origin rpy="0 0 0" xyz="0 0 0.0584" />
         <axis xyz="0 -1 0" />

File: hts_moveit_config/config/fr3.ros2_control.xacro (robot description, xacro)
@@ -1,5 +1,5 @@
 <?xml version="1.0"?>
 <robot xmlns:xacro="http://www.ros.org/wiki/xacro">
-    <xacro:macro name="panda_ros2_control" params="name initial_positions_file ros2_control_hardware_type">
+    <xacro:macro name="fr3_ros2_control" params="name initial_positions_file ros2_control_hardware_type">
         <xacro:property name="initial_positions" value="${xacro.load_yaml(initial_positions_file)['initial_positions']}"/>
         <ros2_control name="${name}" type="system">

File: hts_moveit_config/config/fr3.urdf.xacro (robot description, xacro)
@@ -4,9 +4,9 @@
     <xacro:arg name="ros2_control_hardware_type" default="mock_components" />
     <!-- Import panda urdf file -->
-    <xacro:include filename="$(find hts_description)/urdf/panda.urdf.xacro" />
+    <xacro:include filename="$(find hts_description)/urdf/fr3.urdf.xacro" />
     <!-- Import panda ros2_control description -->
-    <xacro:include filename="panda.ros2_control.xacro" />
+    <xacro:include filename="fr3.ros2_control.xacro" />
     <xacro:include filename="fr3_hand.ros2_control.xacro" />
-    <xacro:panda_ros2_control name="PandaFakeSystem" initial_positions_file="$(arg initial_positions_file)" ros2_control_hardware_type="$(arg ros2_control_hardware_type)"/>
+    <xacro:fr3_ros2_control name="PandaFakeSystem" initial_positions_file="$(arg initial_positions_file)" ros2_control_hardware_type="$(arg ros2_control_hardware_type)"/>
     <xacro:fr3_hand_ros2_control name="PandaHandFakeSystem" ros2_control_hardware_type="$(arg ros2_control_hardware_type)"/>
 </robot>

File: hts_moveit_config/config/fr3_arm.srdf.xacro (robot description, xacro)
@@ -5,5 +5,5 @@
 -->
 <robot xmlns:xacro="http://www.ros.org/wiki/xacro" name="panda">
-  <xacro:include filename="$(find moveit_resources_panda_moveit_config)/config/fr3_arm.xacro" />
+  <xacro:include filename="$(find hts_moveit_config)/config/fr3_arm.xacro" />
   <xacro:fr3_arm />
 </robot>

File: hts_moveit_config/config/fr3_arm_hand.srdf.xacro (robot description, xacro)
@@ -5,6 +5,6 @@
 -->
 <robot xmlns:xacro="http://www.ros.org/wiki/xacro" name="panda">
-  <xacro:include filename="$(find moveit_resources_panda_moveit_config)/config/fr3_arm.xacro" />
-  <xacro:include filename="$(find moveit_resources_panda_moveit_config)/config/hand.xacro" />
+  <xacro:include filename="$(find hts_moveit_config)/config/fr3_arm.xacro" />
+  <xacro:include filename="$(find hts_moveit_config)/config/hand.xacro" />
   <xacro:fr3_arm />
   <xacro:hand />
@@ -33,11 +33,11 @@
   <disable_collisions link1="fr3_hand" link2="fr3_link6" reason="Never" />
   <disable_collisions link1="fr3_hand" link2="fr3_link7" reason="Adjacent" />
-  <disable_collisions link1="panda_leftfinger" link2="fr3_link3" reason="Never" />
-  <disable_collisions link1="panda_leftfinger" link2="fr3_link4" reason="Never" />
-  <disable_collisions link1="panda_leftfinger" link2="fr3_link6" reason="Never" />
-  <disable_collisions link1="panda_leftfinger" link2="fr3_link7" reason="Never" />
-  <disable_collisions link1="fr3_link3" link2="panda_rightfinger" reason="Never" />
-  <disable_collisions link1="fr3_link4" link2="panda_rightfinger" reason="Never" />
-  <disable_collisions link1="fr3_link6" link2="panda_rightfinger" reason="Never" />
-  <disable_collisions link1="fr3_link7" link2="panda_rightfinger" reason="Never" />
+  <disable_collisions link1="fr3_leftfinger" link2="fr3_link3" reason="Never" />
+  <disable_collisions link1="fr3_leftfinger" link2="fr3_link4" reason="Never" />
+  <disable_collisions link1="fr3_leftfinger" link2="fr3_link6" reason="Never" />
+  <disable_collisions link1="fr3_leftfinger" link2="fr3_link7" reason="Never" />
+  <disable_collisions link1="fr3_link3" link2="fr3_rightfinger" reason="Never" />
+  <disable_collisions link1="fr3_link4" link2="fr3_rightfinger" reason="Never" />
+  <disable_collisions link1="fr3_link6" link2="fr3_rightfinger" reason="Never" />
+  <disable_collisions link1="fr3_link7" link2="fr3_rightfinger" reason="Never" />
 </robot>

File: hts_moveit_config/config/hand.xacro (robot description, xacro)
@@ -9,6 +9,6 @@
     <group name="hand">
       <link name="fr3_hand" />
-      <link name="panda_leftfinger" />
-      <link name="panda_rightfinger" />
+      <link name="fr3_leftfinger" />
+      <link name="fr3_rightfinger" />
       <joint name="fr3_finger_joint1" />
       <passive_joint name="fr3_finger_joint2" />
@@ -17,7 +17,7 @@
     <!--END EFFECTOR: Purpose: Represent information about an end effector.-->
     <!--DISABLE COLLISIONS: By default it is assumed that any link of the robot could potentially come into collision with any other link in the robot. This tag disables collision checking between a specified pair of links. -->
-    <disable_collisions link1="fr3_hand" link2="panda_leftfinger" reason="Adjacent" />
-    <disable_collisions link1="fr3_hand" link2="panda_rightfinger" reason="Adjacent" />
-    <disable_collisions link1="panda_leftfinger" link2="panda_rightfinger" reason="Default" />
+    <disable_collisions link1="fr3_hand" link2="fr3_leftfinger" reason="Adjacent" />
+    <disable_collisions link1="fr3_hand" link2="fr3_rightfinger" reason="Adjacent" />
+    <disable_collisions link1="fr3_leftfinger" link2="fr3_rightfinger" reason="Default" />
   </xacro:macro>
 </robot>
